File: smoothie_sd.kicad_pcb (KiCad board)
At the start: 2 copper layers, 41 x 41 mm, 7 parts, among them P1 CONN_02X04

Commit message: gerber
Other:
- board text added: "http://smoothieware.org/"
Changed lines of the file:
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@@
     (area 96.013001 63.55805 171.285715 120.700001)
     (thickness 1.6)
-    (drawings 13)
+    (drawings 14)
     (tracks 71)
     (zones 0)
@@
     (visible_elements 7FFFFFFF)
     (pcbplotparams
-      (layerselection 0x010f8_80000001)
+      (layerselection 0x010f0_80000001)
       (usegerberextensions true)
-      (usegerberattributes true)
       (excludeedgelayer true)
-      (linewidth 0.100000)
+      (linewidth 0.020000)
       (plotframeref false)
       (viasonmask false)
@@
       (psa4output false)
       (plotreference true)
-      (plotvalue true)
+      (plotvalue false)
       (plotinvisibletext false)
       (padsonsilk false)
@@
       (drillshape 0)
       (scaleselection 1)
-      (outputdirectory ""))
+      (outputdirectory gerber/))
   )
   (net 0 "")
@@
     (fp_line (start 0.35052 0.89916) (end 0.7493 1.89992) (layer F.SilkS) (width 0.15))
   )
+  (gr_text http://smoothieware.org/ (at 145.923 90.424 270) (layer F.SilkS)
+    (effects (font (size 1.2 1.2) (thickness 0.2)))
+  )
   (gr_text "by Laurent Le Goff" (at 110.236 91.059 270) (layer F.SilkS)
